Commit message: Changed sensor placement for kinect in the middle, added minimal_ns.launch and robot_ns.launch.xml

File: turtlebot_description/urdf/turtlebot_properties.urdf.xacro (robot description, xacro)
@@ -19,5 +19,5 @@
      (currently in development and awaiting feedback)
    -->
-	<xacro:property name="cam_px" value="-0.087" />
+	<xacro:property name="cam_px" value="0.02" />
 <!--	<xacro:property name="cam_py" value="-0.0125" /> Y varies for different configurations. get sets in sensors_urdf -->
 	<xacro:property name="cam_pz" value="0.2870" />
